File: pork-chop/kicad/pork-chop-control.kicad_pcb (KiCad board)
At the start: 2 copper layers, 88 x 71 mm, 35 parts, among them J1 MUSBD111M0, J2 left, J3 right, SW1 RESET, U1 ATmega32U2, U2 USBLC6-2SC6, Y1 16MHz

Commit message: routing
Parts:
- removed the REF** at (89.0, 106.0)
- moved REF** 35.1 mm to (125.0, 116.0)
- moved R1 9.50 mm to (135.0, 79.5)
- moved J1 7.81 mm to (125.0, 63.0)
- moved C1 7.64 mm to (140.0, 79.5)
- moved R2 7.52 mm to (137.5, 79.5)
- moved SW1 7.52 mm to (139.5, 87.9)
- moved C7 7.43 mm to (113.5, 75.0)
- moved C8 7.17 mm to (121.0, 75.0)
- moved R4 6.80 mm to (118.5, 75.0)
- moved TP5 6.80 mm to (106.5, 76.0)
- moved FB1 6.40 mm to (116.0, 75.0), turned to -90 degrees
- moved J2 5.83 mm to (117.7, 113.1)
- moved J3 5.83 mm to (132.3, 102.9)
- moved H1 5.66 mm to (146.0, 64.0)
- moved FB2 5.15 mm to (117.5, 78.5)
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Routing:
- net GNDPWR: track 51.1 -> 20.1 mm, vias 0 -> 1
- net R2: track 26.3 -> 34.4 mm
- net R3: track 21.2 -> 27.9 mm
- net R4: track 31.9 -> 37.6 mm
- net R0: track 33.8 -> 39.1 mm
- net +5V: track 81.7 -> 86.7 mm
- net Net-(J1-Pad3): track 6.75 -> 9.83 mm
- net /D-: track 4.50 -> 7.52 mm
- net C0: track 26.8 -> 29.6 mm
- net GND: track 21.9 -> 19.3 mm, vias 3 -> 9
- net C4: track 15.6 -> 17.8 mm
- net C9: track 31.0 -> 29.0 mm
- net C1: track 39.6 -> 41.4 mm
- net Net-(FB2-Pad2): track 18.6 -> 20.4 mm
- net Net-(C1-Pad1): track 6.83 -> 5.03 mm
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- added copper zone on B.Cu, net GNDPWR
- added copper zone on F.Cu, net GNDPWR
Other:
- board size 88 x 71 mm -> 50 x 60 mm

Commit message: Silk screen
Connections:
- FL1 pad 4: /D+ -> /D_P
- J1 pad 3: Net-(J1-Pad3) -> /D+
- U2 pad 1: /D+ -> /D_P
- U2 pad 6: Net-(J1-Pad3) -> /D+
Routing:
- net Net-(J1-Pad3): track 9.83 -> 0.00 mm
- net /D_P: track 0.00 -> 4.95 mm
- net /D+: track 4.95 -> 9.83 mm
Other:
- board text added: "The Pork Chop"
- board text added: "jpsecher 2022 v1"

Commit message: move programming pads
Parts:
- added SW2: DEBUG, Button_Switch_SMD:SW_SPST_EVQQ2, F.Cu at (142.5, 91.0)
- J2: value left -> LEFT
- J3: value right -> RIGHT
- TP1: value ~{reset} -> ~{RESET}
- TP3: value MOSI -> PDI
- TP4: value MISO -> PDO
- moved TP4 19.1 mm to (121.0, 112.0)
- moved TP3 19.1 mm to (121.0, 110.0), turned to 180 degrees
- moved TP2 19.0 mm to (121.0, 108.0)
- moved SW1 6.18 mm to (142.5, 82.5), turned to 180 degrees
- moved C1 4.61 mm to (139.0, 75.0)
- moved R1 4.61 mm to (134.0, 75.0)
- moved R2 4.61 mm to (136.5, 75.0)
- moved TP1 0.50 mm to (133.5, 89.0)
Routing:
- net R3: track 27.9 -> 54.3 mm, vias 0 -> 1
- net C8: track 29.8 -> 47.4 mm, vias 0 -> 2
- net C2: track 36.9 -> 20.8 mm
- net GNDPWR: track 20.1 -> 5.16 mm, vias 1 -> 2
- net C3: track 35.7 -> 22.0 mm
- net C1: track 41.4 -> 27.8 mm
- net Net-(R2-Pad2): track 19.1 -> 28.9 mm
- net GND: track 19.1 -> 26.8 mm, vias 9 -> 14
- net C9: track 29.0 -> 31.7 mm
- net +5V: track 86.7 -> 89.2 mm
- net R1: track 37.5 -> 39.6 mm
- net C7: track 23.7 -> 25.3 mm
- net C4: track 17.8 -> 17.0 mm
- net C6: track 24.6 -> 25.4 mm
- net R4: track 37.6 -> 38.2 mm
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
Commit message: Newest layout
Parts:
- moved R5 1.00 mm to (125.0, 81.5)
- moved R6 1.00 mm to (125.0, 79.5)
Connections:
- net /D_P renamed /DD-
- net Net-(FL1-Pad1) renamed /DD+
- R5 pad 2: Dpos -> DDD-
- R6 pad 2: Dneg -> DDD+
- U1 pad 29: Dpos -> DDD+
- U1 pad 30: Dneg -> DDD-
- U2 pad 4: /D- -> /D+
- U2 pad 6: /D+ -> /D-
Routing:
- net Dneg: track 9.33 -> 0.00 mm
- net DDD+: track 0.00 -> 8.87 mm
- net Dpos: track 6.42 -> 0.00 mm
- net DDD-: track 0.00 -> 6.33 mm
- net Net-(FL1-Pad3): track 2.73 -> 3.73 mm
- net Net-(FL1-Pad2): track 2.73 -> 3.73 mm
- net /D+: track 9.83 -> 9.14 mm
- net GNDPWR: vias 2 -> 0
