File: pork-chop/kicad/pork-chop-control.kicad_sch (KiCad schematic)
At the start: 31 parts, among them J1 MUSBD111M0, J2 left, J3 right, SW1 RESET, U1 ATmega32U2, U2 USBLC6-2SC6

Commit message: Silk screen
Connections:
- net D+: now also J1.3 (D+), U2.6 (I/O1); no longer FL1.4, U2.1 (I/O1)
- new net D_P: FL1.4, U2.1 (I/O1)
Changed lines of the file:
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@@
     (stroke (width 0) (type default) (color 0 0 0 0))
   )
-  (label "D+" (at 215.9 60.325 0)
+  (label "D_P" (at 215.9 60.325 0)
     (effects (font (size 1.27 1.27)) (justify left bottom))
   )
@@
     (effects (font (size 1.27 1.27)) (justify left bottom))
   )
-  (label "D+" (at 179.705 65.405 0)
+  (label "D+" (at 175.895 60.325 0)
     (effects (font (size 1.27 1.27)) (justify left bottom))
   )
+  (label "D_P" (at 179.705 65.405 0)
+    (effects (font (size 1.27 1.27)) (justify left bottom))
+  )

Commit message: move programming pads
Parts:
- added SW2: DEBUG, Button_Switch_SMD:SW_SPST_EVQQ2, symbol Switch:SW_Push
- added Y1: 16MHz, Crystal:Crystal_SMD_HC49-SD, symbol Device:Crystal
- J2: value left -> LEFT
- J3: value right -> RIGHT
- TP1: value ~{reset} -> ~{RESET}
- TP3: value MOSI -> PDI
- TP4: value MISO -> PDO
Connections:
- net C8: now also SW2.1
- net R3: now also SW2.2
- net at C2.1, U1.1 (XTAL1): now also Y1.1
- net at C3.1, U1.2 (PC0/XTAL2): now also Y1.2
- no-connect marks 3 -> 5

Commit message: Newest layout
Parts:
- C6: footprint Capacitor_SMD:C_1206_3216Metric_Pad1.33x1.80mm_HandSolder -> Capacitor_SMD:C_0805_2012Metric_Pad1.18x1.45mm_HandSolder
Connections:
- net D+: now also U2.4 (I/O2); no longer U2.6 (I/O1)
- net D-: now also U2.6 (I/O1); no longer U2.4 (I/O2)
- net DD+: now reaches FL1.1, U2.3 (I/O2)
- net D_P renamed DD-
- net Dneg renamed DDD+
- net DDD+: now also U1.29 (D+); no longer U1.30 (D-)
- net Dpos renamed DDD-
- net DDD-: now also U1.30 (D-); no longer U1.29 (D+)
Other:
- moved on the sheet: FL1, R5, R6, U2
