File: pork-chop/kicad/pork-chop.kicad_sch (KiCad schematic)
At the start: 115 parts, among them J1 USB_B_Micro, SW48 Q, SW49 RESET, U1 USBLC6-2SC6, U2 ATmega32U2-A, Y1 16MHz

Commit message: before reorder
Parts:
- removed J1: USB_B_Micro, symbol Connector:USB_B_Micro
- added H10, H2, H3, H4, H5, H6, H7, H8, H9: MountingHole, MountingHole:MountingHole_3.2mm_M3, symbol Mechanical:MountingHole
- H1: footprint (none) -> MountingHole:MountingHole_3.2mm_M3_ISO14580_Pad
- J1: renamed from J?; value USB_C_Receptacle_USB2.0 -> USB_C
- gave numbers to parts that had none: 86
Connections:
- net D+: now also J1.A6 (D+), J1.B6 (D+), U1.3 (I/O2); no longer U1.6 (I/O1)
- net D-: now also J1.A7 (D-), J1.B7 (D-), U1.6 (I/O1); no longer U1.4 (I/O2)
- net DD+: now also U1.4 (I/O2); no longer U1.1 (I/O1)
- net DD-: now also U1.1 (I/O1); no longer U1.3 (I/O2)
- net GND: now also C1.1, J1.A1 (GND), J1.A12 (GND), J1.B1 (GND), J1.B12 (GND); no longer C1.2
- net GNDPWR: now also J1.S1 (SHIELD)
- net at J1.A4 (VBUS), J1.A9 (VBUS), J1.B4 (VBUS)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: now also FB2.1, U1.5 (VBUS)
- net at FB2.2: now also C1.2, F1.1; no longer U1.5 (VBUS)
Other:
- moved on the sheet: C1, C2, D1, D10, D11, D12, D13, D14, D15, D16, D17, D18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
