File: acacia/kicad/controller.kicad_sch (KiCad schematic)
At the start: 33 parts, among them J1 MUSBD111M0, J2 LEFT, J3 RIGHT, SW1 RESET, SW2 DEBUG, U1 ATmega32U2, U2 USBLC6-2SC6, Y1 16MHz

Commit message: rearrange
Parts:
- removed FL1: NCC0805F900KTRF, Inductor_SMD:L_CommonModeChoke_Coilcraft_0805USB, symbol pork-chop-control:Filter_EMI_CommonMode
- added FL1: NCC0805F900KTRF, Inductor_SMD:L_CommonModeChoke_Coilcraft_0805USB, symbol mech-kbd:Filter_EMI_CommonMode
Connections:
- net DD+: now also FL1.1
- net DD-: now also FL1.4
- net at R6.1: now also FL1.2
- net at R5.1: now also FL1.3
Changed lines of the file:
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@@
     (pin "1")
   )
-  (symbol (lib_id "pork-chop-control:Filter_EMI_CommonMode") (at 229.87 65.405 0) (mirror x) (unit 1)
-    (in_bom yes) (on_board yes) (fields_autoplaced)
-    (property "Reference" "FL1" (id 0) (at 229.489 57.15 0))
-    (property "Value" "NCC0805F900KTRF" (id 1) (at 229.489 59.69 0))
+  (symbol (lib_id "power:+5V") (at 78.105 42.545 0) (unit 1)
+    (in_bom yes) (on_board yes) (fields_autoplaced)
+    (property "Reference" "#PWR011" (id 0) (at 78.105 46.355 0)
+      (effects (font (size 1.27 1.27)) hide)
+    )
+    (property "Value" "+5V" (id 1) (at 78.105 36.83 0))
+    (property "Footprint" "" (id 2) (at 78.105 42.545 0)
+      (effects (font (size 1.27 1.27)) hide)
+    )
+    (property "Datasheet" "" (id 3) (at 78.105 42.545 0)
+      (effects (font (size 1.27 1.27)) hide)
+    )
+    (pin "1")
+  )
+  (symbol (lib_id "power:GND") (at 151.13 50.165 0) (unit 1)
+    (in_bom yes) (on_board yes) (fields_autoplaced)
+    (property "Reference" "#PWR014" (id 0) (at 151.13 56.515 0)
+      (effects (font (size 1.27 1.27)) hide)
+    )
+    (property "Value" "GND" (id 1) (at 151.13 55.245 0))
+    (property "Footprint" "" (id 2) (at 151.13 50.165 0)
+      (effects (font (size 1.27 1.27)) hide)
+    )
+    (property "Datasheet" "" (id 3) (at 151.13 50.165 0)
+      (effects (font (size 1.27 1.27)) hide)
+    )
+    (pin "1")
+  )
+  (symbol (lib_id "Connector:TestPoint_Alt") (at 112.395 71.12 0) (unit 1)
+    (in_bom yes) (on_board yes)
+    (property "Reference" "TP3" (id 0) (at 111.125 65.405 0)
+      (effects (font (size 1.27 1.27)) (justify left))
+    )
+    (property "Value" "PDI" (id 1) (at 110.49 63.5 0)
+      (effects (font (size 1.27 1.27)) (justify left))
+    )
+    (property "Footprint" "TestPoint:TestPoint_Pad_1.0x1.0mm" (id 2) (at 117.475 71.12 0)
+      (effects (font (size 1.27 1.27)) hide)
+    )
+    (property "Datasheet" "~" (id 3) (at 117.475 71.12 0)
+      (effects (font (size 1.27 1.27)) hide)
+    )
+    (pin "1")
+  )
+  (symbol (lib_id "power:GND") (at 42.545 86.36 0) (unit 1)
+    (in_bom yes) (on_board yes) (fields_autoplaced)
+    (property "Reference" "#PWR04" (id 0) (at 42.545 92.71 0)
+      (effects (font (size 1.27 1.27)) hide)
+    )
+    (property "Value" "GND" (id 1) (at 42.545 91.44 0))
+    (property "Footprint" "" (id 2) (at 42.545 86.36 0)
+      (effects (font (size 1.27 1.27)) hide)
+    )
+    (property "Datasheet" "" (id 3) (at 42.545 86.36 0)
+      (effects (font (size 1.27 1.27)) hide)
+    )
+    (pin "1")
+  )
+  (symbol (lib_id "power:+5V") (at 29.845 36.83 0) (unit 1)
+    (in_bom yes) (on_board yes) (fields_autoplaced)
+    (property "Reference" "#PWR01" (id 0) (at 29.845 40.64 0)
+      (effects (font (size 1.27 1.27)) hide)
+    )
+    (property "Value" "+5V" (id 1) (at 29.845 31.75 0))
+    (property "Footprint" "" (id 2) (at 29.845 36.83 0)
+      (effects (font (size 1.27 1.27)) hide)
+    )
+    (property "Datasheet" "" (id 3) (at 29.845 36.83 0)
+      (effects (font (size 1.27 1.27)) hide)
+    )
+    (pin "1")
+  )
+  (symbol (lib_id "Connector:TestPoint_Alt") (at 102.87 68.58 0) (unit 1)
+    (in_bom yes) (on_board yes)
+    (property "Reference" "TP2" (id 0) (at 102.235 62.865 0)
+      (effects (font (size 1.27 1.27)) (justify left))
+    )
+    (property "Value" "SCK" (id 1) (at 101.6 60.96 0)
+      (effects (font (size 1.27 1.27)) (justify left))
+    )
+    (property "Footprint" "TestPoint:TestPoint_Pad_1.0x1.0mm" (id 2) (at 107.95 68.58 0)
+      (effects (font (size 1.27 1.27)) hide)
+    )
+    (property "Datasheet" "~" (id 3) (at 107.95 68.58 0)
+      (effects (font (size 1.27 1.27)) hide)
+    )
+    (pin "1")
+  )
+  (symbol (lib_id "mech-kbd:Filter_EMI_CommonMode") (at 229.87 65.405 0) (mirror x) (unit 1)
+    (in_bom yes) (on_board yes)
+    (property "Reference" "FL1" (id 0) (at 229.87 60.325 0))
+    (property "Value" "NCC0805F900KTRF" (id 1) (at 229.235 69.85 0))
     (property "Footprint" "Inductor_SMD:L_CommonModeChoke_Coilcraft_0805USB" (id 2) (at 229.87 66.421 0)
       (effects (font (size 1.27 1.27)) hide)
@@
     (pin "3")
     (pin "4")
-  )
-  (symbol (lib_id "power:+5V") (at 78.105 42.545 0) (unit 1)
-    (in_bom yes) (on_board yes) (fields_autoplaced)
-    (property "Reference" "#PWR011" (id 0) (at 78.105 46.355 0)
-      (effects (font (size 1.27 1.27)) hide)
-    )
-    (property "Value" "+5V" (id 1) (at 78.105 36.83 0))
-    (property "Footprint" "" (id 2) (at 78.105 42.545 0)
-      (effects (font (size 1.27 1.27)) hide)
-    )
-    (property "Datasheet" "" (id 3) (at 78.105 42.545 0)
-      (effects (font (size 1.27 1.27)) hide)
-    )
-    (pin "1")
-  )
-  (symbol (lib_id "power:GND") (at 151.13 50.165 0) (unit 1)
-    (in_bom yes) (on_board yes) (fields_autoplaced)
-    (property "Reference" "#PWR014" (id 0) (at 151.13 56.515 0)
-      (effects (font (size 1.27 1.27)) hide)
-    )
-    (property "Value" "GND" (id 1) (at 151.13 55.245 0))
-    (property "Footprint" "" (id 2) (at 151.13 50.165 0)
-      (effects (font (size 1.27 1.27)) hide)
-    )
-    (property "Datasheet" "" (id 3) (at 151.13 50.165 0)
-      (effects (font (size 1.27 1.27)) hide)
-    )
-    (pin "1")
-  )
-  (symbol (lib_id "Connector:TestPoint_Alt") (at 112.395 71.12 0) (unit 1)
-    (in_bom yes) (on_board yes)
-    (property "Reference" "TP3" (id 0) (at 111.125 65.405 0)
-      (effects (font (size 1.27 1.27)) (justify left))
-    )
-    (property "Value" "PDI" (id 1) (at 110.49 63.5 0)
-      (effects (font (size 1.27 1.27)) (justify left))
-    )
-    (property "Footprint" "TestPoint:TestPoint_Pad_1.0x1.0mm" (id 2) (at 117.475 71.12 0)
-      (effects (font (size 1.27 1.27)) hide)
-    )
-    (property "Datasheet" "~" (id 3) (at 117.475 71.12 0)
-      (effects (font (size 1.27 1.27)) hide)
-    )
-    (pin "1")
-  )
-  (symbol (lib_id "power:GND") (at 42.545 86.36 0) (unit 1)
-    (in_bom yes) (on_board yes) (fields_autoplaced)
-    (property "Reference" "#PWR04" (id 0) (at 42.545 92.71 0)
-      (effects (font (size 1.27 1.27)) hide)
-    )
-    (property "Value" "GND" (id 1) (at 42.545 91.44 0))
-    (property "Footprint" "" (id 2) (at 42.545 86.36 0)
-      (effects (font (size 1.27 1.27)) hide)
-    )
-    (property "Datasheet" "" (id 3) (at 42.545 86.36 0)
-      (effects (font (size 1.27 1.27)) hide)
-    )
-    (pin "1")
-  )
-  (symbol (lib_id "power:+5V") (at 29.845 36.83 0) (unit 1)
-    (in_bom yes) (on_board yes) (fields_autoplaced)
-    (property "Reference" "#PWR01" (id 0) (at 29.845 40.64 0)
-      (effects (font (size 1.27 1.27)) hide)
-    )
-    (property "Value" "+5V" (id 1) (at 29.845 31.75 0))
-    (property "Footprint" "" (id 2) (at 29.845 36.83 0)
-      (effects (font (size 1.27 1.27)) hide)
-    )
-    (property "Datasheet" "" (id 3) (at 29.845 36.83 0)
-      (effects (font (size 1.27 1.27)) hide)
-    )
-    (pin "1")
-  )
-  (symbol (lib_id "Connector:TestPoint_Alt") (at 102.87 68.58 0) (unit 1)
-    (in_bom yes) (on_board yes)
-    (property "Reference" "TP2" (id 0) (at 102.235 62.865 0)
-      (effects (font (size 1.27 1.27)) (justify left))
-    )
-    (property "Value" "SCK" (id 1) (at 101.6 60.96 0)
-      (effects (font (size 1.27 1.27)) (justify left))
-    )
-    (property "Footprint" "TestPoint:TestPoint_Pad_1.0x1.0mm" (id 2) (at 107.95 68.58 0)
-      (effects (font (size 1.27 1.27)) hide)
-    )
-    (property "Datasheet" "~" (id 3) (at 107.95 68.58 0)
-      (effects (font (size 1.27 1.27)) hide)
-    )
-    (pin "1")
   )
   (symbol (lib_id "Device:C") (at 151.13 45.72 0) (unit 1)
@@
       (reference "FB2") (unit 1) (value "120") (footprint "Resistor_SMD:R_0805_2012Metric_Pad1.20x1.40mm_HandSolder")
     )
-    (path "/64e37c6b-f3b1-4687-95af-e8f3de831990"
+    (path "/9a5eb83c-2ffe-44ed-b17b-3c2114c6e8e2"
       (reference "FL1") (unit 1) (value "NCC0805F900KTRF") (footprint "Inductor_SMD:L_CommonModeChoke_Coilcraft_0805USB")
     )
