File: acacia/kicad/acacia.kicad_pcb (KiCad board)
At the start: 2 copper layers, 274 x 158 mm, 122 parts, among them J1 USB4500-03-0-A, SW1 A, SW10 C, SW11 R, SW12 F, SW13 V, SW14 T, SW15 G, SW16 Back, SW17 Gui, SW18 Ctl, SW19 Alt, SW2 Z, SW20 Sft, SW21 Fwd, SW22 AltGr, SW23 L1, SW24 L2, SW25 Ctl, SW26 U, SW27 J, SW28 M, SW29 H, SW3 Esc, SW30 N, SW31 I, SW32 K, SW33 Comm, SW34 O, SW35 L, SW36 Dot, SW38 P, SW39 Semi, SW4 B, SW40 Slsh, SW41 Y, SW42 Png, SW43 QMK, SW48 Q, SW49 RESET, SW5 W, SW6 S, SW7 X, SW8 E, SW9 D, U1 USBLC6-2SC6, U2 ATmega32U2-A, Y1 16MHz

Commit message: keys layed out
Parts:
- added TP3: D0, TestPoint:TestPoint_Pad_1.0x1.0mm, B.Cu at (78.0, 164.0)
- added TP4: D1, TestPoint:TestPoint_Pad_1.0x1.0mm, B.Cu at (74.9, 164.0)
- added TP5: C2, TestPoint:TestPoint_Pad_1.0x1.0mm, B.Cu at (71.9, 164.0)
- added TP6: C4, TestPoint:TestPoint_Pad_1.0x1.0mm, B.Cu at (74.9, 167.1)
- added TP7: C5, TestPoint:TestPoint_Pad_1.0x1.0mm, B.Cu at (78.0, 167.1)
- C1, C2, C3, C4, C5, C6, C7, C8, D1, D10, D11, D12, D13, D14, D15, D16, D17, D18, D19, D2, D20, D21, D22, D23, D24, D25, D26, D27, D28, D29, D3, D30, D31, D32, D33, D34, D35, D36, D37, D38, D39, D4, D40, D41, D48, D5, D6, D7, D8, D9, F1, FB1, FB2, FL1, R1, R2, R3, R4, R5, R6, R7, R8, SW43, SW49, TP1, TP2, U1, U2: moved to B.Cu
- Y1: footprint mech-kbd:MX-Hotswap-1.5U -> Crystal:Crystal_SMD_HC49-SD; moved to B.Cu
- moved SW40 418.5 mm to (271.0, 102.5), turned to 15 degrees
- moved D30 375.1 mm to (282.8, 93.0), turned to 180 degrees
- moved SW23 374.7 mm to (202.0, 136.5), turned to -45 degrees
- moved SW30 374.7 mm to (287.0, 88.2), turned to 15 degrees
- moved SW35 368.3 mm to (241.5, 74.5), turned to 20 degrees
- moved SW27 353.6 mm to (205.0, 89.2), turned to 25 degrees
- moved SW39 350.6 mm to (266.0, 84.0), turned to 15 degrees
- moved D38 346.4 mm to (261.2, 88.5), turned to 180 degrees
- moved SW24 345.0 mm to (188.9, 151.3), turned to -38 degrees
- moved SW32 344.5 mm to (220.0, 75.0), turned to 23 degrees
- moved D41 339.1 mm to (273.2, 73.8), turned to 180 degrees
- moved SW25 336.0 mm to (178.0, 168.5), turned to -29 degrees
- moved SW33 334.0 mm to (227.4, 92.5), turned to 23 degrees
- moved D34 333.6 mm to (229.0, 62.0), turned to 180 degrees
- moved SW49 328.1 mm to (174.1, 130.0), turned to 180 degrees
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Connections:
- U2 pad 25: unconnected-(U2-Pad25) -> Net-(U2-Pad25)
- U2 pad 26: unconnected-(U2-Pad26) -> Net-(U2-Pad26)
- U2 pad 5: unconnected-(U2-Pad5) -> Net-(U2-Pad5)
- U2 pad 6: unconnected-(U2-Pad6) -> Net-(U2-Pad6)
- U2 pad 7: unconnected-(U2-Pad7) -> Net-(U2-Pad7)

Commit message: wip
Parts:
- removed TP1: GND, TestPoint:TestPoint_Pad_1.0x1.0mm
- removed TP2: 5V, TestPoint:TestPoint_Pad_1.0x1.0mm
- removed TP3: D0, TestPoint:TestPoint_Pad_1.0x1.0mm
- removed TP4: D1, TestPoint:TestPoint_Pad_1.0x1.0mm
- removed TP5: C2, TestPoint:TestPoint_Pad_1.0x1.0mm
- removed TP6: C4, TestPoint:TestPoint_Pad_1.0x1.0mm
- removed TP7: C5, TestPoint:TestPoint_Pad_1.0x1.0mm
- J1: moved to B.Cu
- moved R2 149.6 mm to (159.8, 91.1), turned to 0 degrees
- moved FB2 147.5 mm to (167.0, 73.0)
- moved U1 145.0 mm to (160.0, 74.0), turned to -90 degrees
- moved R5 144.6 mm to (147.2, 113.2)
- moved R3 140.4 mm to (159.8, 93.1)
- moved U2 135.9 mm to (159.0, 113.0)
- moved R7 134.0 mm to (149.0, 64.2)
- moved R6 133.1 mm to (153.8, 102.0), turned to 0 degrees
- moved R4 131.5 mm to (147.5, 116.1)
- moved R1 121.7 mm to (155.0, 75.0)
- moved Y1 115.8 mm to (170.0, 110.4), turned to -90 degrees
- moved C1 69.5 mm to (174.0, 71.8)
- moved F1 58.7 mm to (174.4, 76.0)
- moved R8 55.8 mm to (172.2, 65.5)
- moved C2 55.2 mm to (149.8, 76.8)
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Connections:
- FL1 pad 1: /DD- -> Net-(FL1-Pad1)
- FL1 pad 2: Net-(FL1-Pad2) -> /DD-
- FL1 pad 3: Net-(FL1-Pad3) -> /DD+
- FL1 pad 4: /DD+ -> Net-(FL1-Pad4)
- R2 pad 1: Net-(FL1-Pad3) -> Net-(FL1-Pad1)
- R2 pad 2: DDD+ -> DDD-
- R3 pad 1: Net-(FL1-Pad2) -> Net-(FL1-Pad4)
- R3 pad 2: DDD- -> DDD+
- U1 pad 1: /DD- -> /D-
- U1 pad 6: /D- -> /DD-
Routing:
- net DDD-: track 0.00 -> 18.8 mm
- net Net-(C3-Pad1): track 0.00 -> 16.1 mm
- net DDD+: track 0.00 -> 16.1 mm
- net Net-(C4-Pad1): track 0.00 -> 14.8 mm
- net Net-(FL1-Pad4): track 0.00 -> 13.9 mm
- net Net-(FL1-Pad1): track 0.00 -> 12.4 mm
- net +5V: track 0.00 -> 9.90 mm
- net /D-: track 0.00 -> 8.21 mm
- net /D+: track 0.00 -> 7.22 mm
- net GND: track 0.00 -> 5.92 mm
- net /DD-: track 0.00 -> 3.41 mm
- net /DD+: track 0.00 -> 3.41 mm
- added copper zone on B.Cu, net GND

Commit message: keys routed
Parts:
- moved D30 99.7 mm to (185.0, 112.5), turned to 90 degrees
- moved D40 95.9 mm to (276.0, 75.0)
- moved D20 21.2 mm to (156.5, 163.0)
- moved SW43 21.2 mm to (137.5, 136.5)
- moved D41 20.4 mm to (280.0, 93.0), turned to 90 degrees
- moved R6 20.1 mm to (158.5, 121.5), turned to -90 degrees
- moved D29 17.9 mm to (178.0, 95.0)
- moved D19 15.3 mm to (128.0, 142.5), turned to -90 degrees
- moved D22 15.0 mm to (218.0, 118.0)
- moved D23 12.9 mm to (202.0, 124.5), turned to -90 degrees
- moved D17 12.1 mm to (86.0, 119.0), turned to 0 degrees
- moved D2 11.7 mm to (46.5, 92.5)
- moved D8 11.0 mm to (93.0, 62.0), turned to 0 degrees
- moved D24 11.0 mm to (179.0, 142.0), turned to -90 degrees
- moved D39 10.7 mm to (260.5, 98.0), turned to 0 degrees
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Connections:
- net DDD+ renamed DDDD+
- net DDD- renamed DDDD-
- FL1 pad 1: Net-(FL1-Pad1) -> /DDD+
- FL1 pad 2: /DD- -> /DD+
- FL1 pad 3: /DD+ -> /DD-
- FL1 pad 4: Net-(FL1-Pad4) -> /DDD-
- R2 pad 1: Net-(FL1-Pad1) -> /DDD-
- R3 pad 1: Net-(FL1-Pad4) -> /DDD+
- SW29 pad 1: Net-(D29-Pad2) -> Net-(D30-Pad2)
- SW30 pad 1: Net-(D30-Pad2) -> Net-(D41-Pad2)
- SW30 pad 2: C6 -> C9
- SW41 pad 1: Net-(D40-Pad2) -> Net-(D29-Pad2)
- SW41 pad 2: C9 -> C6
- SW42 pad 1: Net-(D41-Pad2) -> Net-(D40-Pad2)
- U1 pad 1: /D- -> /D+
- U1 pad 3: /D+ -> /D-
- U1 pad 4: /DD+ -> /DD-
- U1 pad 6: /DD- -> /DD+
- U2 pad 19: C5 -> R0
- U2 pad 8: R0 -> C5
Routing:
- net R3: track 0.00 -> 418.9 mm, vias 0 -> 5
- net R0: track 0.00 -> 417.7 mm, vias 0 -> 10
- net R4: track 0.00 -> 384.1 mm, vias 0 -> 5
- net R1: track 0.00 -> 351.5 mm, vias 0 -> 13
- net R2: track 0.00 -> 318.8 mm, vias 0 -> 12
- net C9: track 0.00 -> 241.2 mm, vias 0 -> 3
- net C0: track 0.00 -> 217.2 mm, vias 0 -> 3
- net C4: track 0.00 -> 189.2 mm
- net C8: track 0.00 -> 180.6 mm, vias 0 -> 2
- net C5: track 0.00 -> 162.1 mm
- net C7: track 0.00 -> 160.9 mm, vias 0 -> 2
- net C6: track 0.00 -> 154.6 mm, vias 0 -> 3
- net C1: track 0.00 -> 139.5 mm, vias 0 -> 2
- net C2: track 0.00 -> 123.4 mm, vias 0 -> 2
- net C3: track 0.00 -> 120.1 mm, vias 0 -> 3
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- added copper zone on F.Cu, net GND

Commit message: routing
Parts:
- added TP1: GND, TestPoint:TestPoint_Pad_1.0x1.0mm, B.Cu at (165.5, 81.5)
- added TP2: 5V, TestPoint:TestPoint_Pad_1.0x1.0mm, B.Cu at (168.6, 81.5)
- added TP3: D0, TestPoint:TestPoint_Pad_1.0x1.0mm, B.Cu at (151.5, 94.5)
- added TP4: D1, TestPoint:TestPoint_Pad_1.0x1.0mm, B.Cu at (151.5, 92.5)
- added TP5: C2, TestPoint:TestPoint_Pad_1.0x1.0mm, B.Cu at (151.5, 96.5)
- added TP6: C4, TestPoint:TestPoint_Pad_1.0x1.0mm, B.Cu at (151.5, 98.5)
- added TP7: C5, TestPoint:TestPoint_Pad_1.0x1.0mm, B.Cu at (151.5, 100.5)
- H1: value case -> MountingHole; footprint MountingHole:MountingHole_3.2mm_M3_ISO14580_Pad -> MountingHole:MountingHole_3.2mm_M3
- SW23: value L1 -> L2
- SW24: value L2 -> L1
- SW29: value H -> N
- SW3: value Esc -> Tab
- SW30: value N -> Enter
- SW41: value Y -> H
- SW42: value Png -> Y
- moved SW43 51.8 mm to (171.0, 97.0)
- moved C2 25.5 mm to (173.5, 67.5), turned to 90 degrees
- moved R8 25.3 mm to (147.0, 67.5), turned to -90 degrees
- moved R1 22.8 mm to (176.5, 67.5), turned to 90 degrees
- moved SW49 12.0 mm to (143.5, 119.0)
- moved C7 6.90 mm to (143.5, 114.0)
- moved C1 6.50 mm to (167.5, 72.0), turned to -90 degrees
- moved R4 6.10 mm to (143.5, 111.5), turned to 0 degrees
- moved FB1 5.84 mm to (173.5, 72.0), turned to 90 degrees
- moved R5 5.67 mm to (143.5, 109.0)
- moved F1 4.07 mm to (170.5, 77.0), turned to -90 degrees
- moved FB2 3.64 mm to (170.5, 72.0), turned to -90 degrees
- moved R7 3.29 mm to (149.5, 67.5), turned to -90 degrees
- moved D24 1.50 mm to (180.5, 142.0)
- moved D29 1.50 mm to (179.5, 95.0)
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Routing:
- net +5V: track 9.90 -> 114.5 mm, vias 0 -> 2
- net /VBUS: track 0.00 -> 32.4 mm, vias 0 -> 2
- net Net-(TP4-Pad1): track 0.00 -> 30.3 mm, vias 0 -> 2
- net Net-(TP3-Pad1): track 0.00 -> 28.0 mm, vias 0 -> 2
- net Net-(TP5-Pad1): track 0.00 -> 25.0 mm, vias 0 -> 2
- net ~{RESET}: track 0.00 -> 24.2 mm, vias 0 -> 2
- net Net-(J1-PadB5): track 0.00 -> 18.6 mm
- net GNDPWR: track 0.00 -> 16.3 mm, vias 0 -> 1
- net GND: track 5.92 -> 20.8 mm, vias 0 -> 12
- net Net-(TP6-Pad1): track 0.00 -> 14.2 mm
- net Net-(J1-PadA5): track 0.00 -> 11.5 mm
- net Net-(TP7-Pad1): track 0.00 -> 11.3 mm
- net Net-(C2-Pad1): track 0.00 -> 5.48 mm
- net Net-(C1-Pad2): track 0.00 -> 5.47 mm
- net Net-(C7-Pad1): track 0.00 -> 5.02 mm
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- added copper zone on F.Cu, net GNDPWR

Commit message: routing done
Parts:
- moved D23 8.50 mm to (193.5, 124.5)
- moved SW49 7.28 mm to (136.5, 121.0)
- moved C7 7.07 mm to (144.5, 121.0), turned to 0 degrees
- moved R4 7.07 mm to (144.5, 118.5), turned to 180 degrees
- moved R5 7.07 mm to (142.5, 116.0)
- moved D24 5.41 mm to (185.0, 139.0)
- moved TP1 3.91 mm to (168.5, 84.0)
- moved D33 3.35 mm to (223.5, 99.0)
- moved D15 2.24 mm to (129.0, 111.0)
- moved SW43 1.00 mm to (171.0, 96.0)
- moved D14 0.50 mm to (131.5, 90.8)
- moved D3 0.50 mm to (35.0, 74.5)
Routing:
- net +5V: track 114.5 -> 108.5 mm
- net C4: track 189.2 -> 184.4 mm
- net C5: track 162.1 -> 166.6 mm
- net C9: track 239.8 -> 235.5 mm
- net Net-(D33-Pad2): track 3.77 -> 7.41 mm
- net GND: track 20.8 -> 17.8 mm, vias 12 -> 17
- net R2: track 319.4 -> 322.2 mm
- net Net-(D15-Pad2): track 11.9 -> 14.3 mm
- net Net-(D23-Pad2): track 5.50 -> 7.57 mm
- net C7: track 160.9 -> 162.9 mm
- net R4: track 384.1 -> 382.6 mm
- net R0: track 418.3 -> 417.2 mm
- net C6: track 155.9 -> 156.9 mm
- net C1: track 139.5 -> 138.7 mm

Commit message: pcb finished
Other:
- board text added: "2022 jpsecher"
- board text added: "Acacia"
