File: acacia/kicad/acacia-2.kicad_sch (KiCad schematic)
At the start: 123 parts, among them J1 GroveMiniTrack, J2 TM040040, J3 USB4105-GF-A-060, SW1 Q, SW10 P, SW11 A, SW12 S, SW13 D, SW14 F, SW15 G, SW16 H, SW17 J, SW18 K, SW19 L, SW2 W, SW20 B, SW21 RESET, SW22 Z, SW23 X, SW24 C, SW25 V, SW26 Sft, SW27 Spc, SW28 N, SW29 M, SW3 E, SW30 Com, SW31 Dot, SW32 Tab, SW33 Prv, SW34 L1, SW35 AGr, SW36 Esc, SW37 Del, SW38 Nxt, SW39 Ent, SW4 R, SW5 T, SW6 Y, SW7 U, SW8 I, SW9 O, U1 ATmega32U4-A, U2 USBLC6-2SC6, Y1 16MHz

Commit message: before reordering
Connections:
- net BTN: now also U1.28 (PB4); no longer U1.1 (PE6)
- net RGB: now also U1.29 (PB5); no longer U1.8 (PB0)
Changed lines of the file:
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@@
   (no_connect (at 240.03 64.77))
   (no_connect (at 269.24 82.55))
+  (no_connect (at 240.03 102.87))
   (no_connect (at 269.24 87.63))
   (no_connect (at 34.925 149.225))
   (no_connect (at 209.55 62.23))
   (no_connect (at 240.03 52.07))
-  (no_connect (at 240.03 57.15))
+  (no_connect (at 240.03 46.99))
   (no_connect (at 65.405 144.145))
   (no_connect (at 269.24 85.09))
@@
   (no_connect (at 167.005 107.315))
   (no_connect (at 269.24 92.71))
-  (no_connect (at 240.03 59.69))
   (no_connect (at 269.24 90.17))
   (no_connect (at 240.03 62.23))
@@
     (stroke (width 0) (type default))
   )
-  (wire (pts (xy 240.03 46.99) (xy 241.935 46.99))
-    (stroke (width 0) (type default))
-  )
   (wire (pts (xy 33.02 80.01) (xy 34.29 80.01))
     (stroke (width 0) (type default))
@@
     (stroke (width 0) (type default))
   )
-  (wire (pts (xy 259.08 82.55) (xy 259.08 80.01))
-    (stroke (width 0) (type default))
-  )
   (wire (pts (xy 67.945 158.115) (xy 67.945 154.305))
     (stroke (width 0) (type default))
@@
     (stroke (width 0) (type default))
   )
-  (wire (pts (xy 249.555 82.55) (xy 259.08 82.55))
-    (stroke (width 0) (type default))
-  )
   (wire (pts (xy 167.64 34.29) (xy 167.64 35.56))
     (stroke (width 0) (type default))
@@
     (stroke (width 0) (type default))
   )
-  (wire (pts (xy 249.555 102.87) (xy 249.555 82.55))
-    (stroke (width 0) (type default))
-  )
   (wire (pts (xy 240.03 72.39) (xy 241.935 72.39))
     (stroke (width 0) (type default))
@@
     (stroke (width 0) (type default))
   )
+  (wire (pts (xy 259.08 80.01) (xy 259.08 57.15))
+    (stroke (width 0) (type default))
+  )
   (wire (pts (xy 224.79 39.37) (xy 224.79 26.67))
     (stroke (width 0) (type default))
@@
     (stroke (width 0) (type default))
   )
+  (wire (pts (xy 240.03 59.69) (xy 241.935 59.69))
+    (stroke (width 0) (type default))
+  )
   (wire (pts (xy 72.39 63.5) (xy 72.39 80.01))
     (stroke (width 0) (type default))
@@
     (stroke (width 0) (type default))
   )
+  (wire (pts (xy 259.08 57.15) (xy 240.03 57.15))
+    (stroke (width 0) (type default))
+  )
   (wire (pts (xy 129.54 41.91) (xy 128.27 41.91))
     (stroke (width 0) (type default))
@@
     (stroke (width 0) (type default))
   )
-  (wire (pts (xy 240.03 102.87) (xy 249.555 102.87))
-    (stroke (width 0) (type default))
-  )
   (wire (pts (xy 34.29 30.48) (xy 34.29 46.99))
     (stroke (width 0) (type default))
@@
     (effects (font (size 1.27 1.27)) (justify left bottom))
   )
-  (label "BTN" (at 251.46 82.55 0) (fields_autoplaced)
+  (label "BTN" (at 251.46 57.15 0) (fields_autoplaced)
     (effects (font (size 1.27 1.27)) (justify left bottom))
   )
@@
     )
   )
-  (global_label "RGB" (shape input) (at 241.935 46.99 0) (fields_autoplaced)
+  (global_label "RGB" (shape input) (at 241.935 59.69 0) (fields_autoplaced)
     (effects (font (size 1.27 1.27)) (justify left))
-    (property "Intersheetrefs" "${INTERSHEET_REFS}" (at 248.6508 46.99 0)
+    (property "Intersheetrefs" "${INTERSHEET_REFS}" (at 248.6508 59.69 0)
       (effects (font (size 1.27 1.27)) (justify left) hide)
     )

Commit message: leds
Parts:
- added C9: 1µ, Capacitor_SMD:C_0805_2012Metric_Pad1.18x1.45mm_HandSolder, symbol Device:C
Connections:
- net +5V: now also C9.1
- net BTN: now also U1.30 (PB6); no longer U1.28 (PB4)
- net C0: now also U1.37 (PF6); no longer U1.25 (PD4)
- net C1: now also U1.39 (PF4); no longer U1.21 (PD3)
- net C2: now also U1.38 (PF5); no longer U1.20 (PD2)
- net C3: now also U1.36 (PF7); no longer U1.32 (PC7)
- net C4: now also U1.32 (PC7); no longer U1.31 (PC6)
- net C5: now also U1.20 (PD2); no longer U1.39 (PF4)
- net C8: now also U1.21 (PD3); no longer U1.40 (PF1)
- net C9: now also U1.22 (PD5); no longer U1.41 (PF0)
- net GNDD: now also C9.2
- net R0: now also U1.40 (PF1); no longer U1.22 (PD5)
- net R1: now also U1.41 (PF0); no longer U1.38 (PF5)
- net R2: now also U1.28 (PB4); no longer U1.37 (PF6)
- net R3: now also U1.25 (PD4); no longer U1.36 (PF7)
- net SCL: no longer J1.3 (Pin_3)
- net SDA: now also J1.3 (Pin_3)
Changed lines of the file:
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@@
   (junction (at 170.18 133.35) (diameter 0) (color 0 0 0 0)
   )
+  (junction (at 233.68 26.67) (diameter 0) (color 0 0 0 0)
+  )
   (junction (at 102.87 87.63) (diameter 0) (color 0 0 0 0)
   )
@@
   (no_connect (at 269.24 92.71))
   (no_connect (at 269.24 90.17))
-  (no_connect (at 240.03 62.23))
+  (no_connect (at 240.03 69.85))
   (no_connect (at 240.03 49.53))
   (no_connect (at 240.03 54.61))
@@
     (stroke (width 0) (type default))
   )
+  (wire (pts (xy 242.57 35.56) (xy 242.57 36.83))
+    (stroke (width 0) (type default))
+  )
   (wire (pts (xy 159.385 114.935) (xy 159.385 116.84))
     (stroke (width 0) (type default))
@@
     (stroke (width 0) (type default))
   )
+  (wire (pts (xy 242.57 26.67) (xy 242.57 27.94))
+    (stroke (width 0) (type default))
+  )
   (wire (pts (xy 215.9 23.495) (xy 215.9 26.67))
     (stroke (width 0) (type default))
@@
     (stroke (width 0) (type default))
   )
+  (wire (pts (xy 233.68 26.67) (xy 242.57 26.67))
+    (stroke (width 0) (type default))
+  )
   (wire (pts (xy 115.57 58.42) (xy 115.57 61.595))
     (stroke (width 0) (type default))
@@
     (stroke (width 0) (type default))
   )
-  (wire (pts (xy 259.08 80.01) (xy 259.08 57.15))
+  (wire (pts (xy 259.08 62.23) (xy 259.08 80.01))
     (stroke (width 0) (type default))
   )
@@
     (stroke (width 0) (type default))
   )
-  (wire (pts (xy 240.03 69.85) (xy 241.935 69.85))
+  (wire (pts (xy 240.03 62.23) (xy 259.08 62.23))
     (stroke (width 0) (type default))
   )
@@
     (stroke (width 0) (type default))
   )
+  (wire (pts (xy 240.03 57.15) (xy 241.935 57.15))
+    (stroke (width 0) (type default))
+  )
   (wire (pts (xy 77.47 58.42) (xy 77.47 61.595))
     (stroke (width 0) (type default))
@@
     (stroke (width 0) (type default))
   )
-  (wire (pts (xy 259.08 57.15) (xy 240.03 57.15))
-    (stroke (width 0) (type default))
-  )
   (wire (pts (xy 129.54 41.91) (xy 128.27 41.91))
     (stroke (width 0) (type default))
@@
     (effects (font (size 1.27 1.27)) (justify left bottom))
   )
-  (label "BTN" (at 251.46 57.15 0) (fields_autoplaced)
+  (label "BTN" (at 251.46 62.23 0) (fields_autoplaced)
     (effects (font (size 1.27 1.27)) (justify left bottom))
   )
@@
     (effects (font (size 1.27 1.27)) (justify left bottom))
   )
-  (label "SCL" (at 256.54 33.02 0) (fields_autoplaced)
+  (label "SDA" (at 256.54 33.02 0) (fields_autoplaced)
     (effects (font (size 1.27 1.27)) (justify left bottom))
   )
@@
     )
   )
-  (global_label "C8" (shape input) (at 241.935 110.49 0) (fields_autoplaced)
+  (global_label "C8" (shape input) (at 241.935 85.09 0) (fields_autoplaced)
     (effects (font (size 1.27 1.27)) (justify left))
-    (property "Intersheetrefs" "${INTERSHEET_REFS}" (at 246.8276 110.4106 0)
+    (property "Intersheetrefs" "${INTERSHEET_REFS}" (at 246.8276 85.0106 0)
       (effects (font (size 1.27 1.27)) (justify left) hide)
     )
@@
     )
   )
-  (global_label "R3" (shape input) (at 241.935 120.65 0) (fields_autoplaced)
+  (global_label "R3" (shape input) (at 241.935 87.63 0) (fields_autoplaced)
     (effects (font (size 1.27 1.27)) (justify left))
-    (property "Intersheetrefs" "${INTERSHEET_REFS}" (at 246.8276 120.7294 0)
+    (property "Intersheetrefs" "${INTERSHEET_REFS}" (at 246.8276 87.7094 0)
       (effects (font (size 1.27 1.27)) (justify left) hide)
     )
@@
     )
   )
-  (global_label "C5" (shape input) (at 241.935 113.03 0) (fields_autoplaced)
+  (global_label "C5" (shape input) (at 241.935 82.55 0) (fields_autoplaced)
     (effects (font (size 1.27 1.27)) (justify left))
-    (property "Intersheetrefs" "${INTERSHEET_REFS}" (at 246.8276 112.9506 0)
+    (property "Intersheetrefs" "${INTERSHEET_REFS}" (at 246.8276 82.4706 0)
       (effects (font (size 1.27 1.27)) (justify left) hide)
     )
@@
     )
   )
-  (global_label "R0" (shape input) (at 241.935 90.17 0) (fields_autoplaced)
+  (global_label "R0" (shape input) (at 241.935 110.49 0) (fields_autoplaced)
     (effects (font (size 1.27 1.27)) (justify left))
-    (property "Intersheetrefs" "${INTERSHEET_REFS}" (at 246.8276 90.2494 0)
+    (property "Intersheetrefs" "${INTERSHEET_REFS}" (at 246.8276 110.5694 0)
       (effects (font (size 1.27 1.27)) (justify left) hide)
     )
   )
-  (global_label "C3" (shape input) (at 241.935 72.39 0) (fields_autoplaced)
+  (global_label "C3" (shape input) (at 241.935 120.65 0) (fields_autoplaced)
     (effects (font (size 1.27 1.27)) (justify left))
-    (property "Intersheetrefs" "${INTERSHEET_REFS}" (at 246.8276 72.3106 0)
+    (property "Intersheetrefs" "${INTERSHEET_REFS}" (at 246.8276 120.5706 0)
       (effects (font (size 1.27 1.27)) (justify left) hide)
     )
   )
-  (global_label "R1" (shape input) (at 241.935 115.57 0) (fields_autoplaced)
+  (global_label "R1" (shape input) (at 241.935 107.95 0) (fields_autoplaced)
     (effects (font (size 1.27 1.27)) (justify left))
-    (property "Intersheetrefs" "${INTERSHEET_REFS}" (at 246.8276 115.6494 0)
+    (property "Intersheetrefs" "${INTERSHEET_REFS}" (at 246.8276 108.0294 0)
       (effects (font (size 1.27 1.27)) (justify left) hide)
     )
@@
     )
   )
-  (global_label "C9" (shape input) (at 241.935 107.95 0) (fields_autoplaced)
+  (global_label "C9" (shape input) (at 241.935 90.17 0) (fields_autoplaced)
     (effects (font (size 1.27 1.27)) (justify left))
-    (property "Intersheetrefs" "${INTERSHEET_REFS}" (at 246.8276 107.8706 0)
+    (property "Intersheetrefs" "${INTERSHEET_REFS}" (at 246.8276 90.0906 0)
       (effects (font (size 1.27 1.27)) (justify left) hide)
     )
@@
     )
   )
-  (global_label "C4" (shape input) (at 241.935 69.85 0) (fields_autoplaced)
+  (global_label "C4" (shape input) (at 241.935 72.39 0) (fields_autoplaced)
     (effects (font (size 1.27 1.27)) (justify left))
-    (property "Intersheetrefs" "${INTERSHEET_REFS}" (at 246.8276 69.7706 0)
+    (property "Intersheetrefs" "${INTERSHEET_REFS}" (at 246.8276 72.3106 0)
       (effects (font (size 1.27 1.27)) (justify left) hide)
     )
   )
-  (global_label "C2" (shape input) (at 241.935 82.55 0) (fields_autoplaced)
+  (global_label "C2" (shape input) (at 241.935 115.57 0) (fields_autoplaced)
     (effects (font (size 1.27 1.27)) (justify left))
-    (property "Intersheetrefs" "${INTERSHEET_REFS}" (at 246.8276 82.4706 0)
+    (property "Intersheetrefs" "${INTERSHEET_REFS}" (at 246.8276 115.4906 0)
       (effects (font (size 1.27 1.27)) (justify left) hide)
     )
@@
     )
   )
-  (global_label "C1" (shape input) (at 241.935 85.09 0) (fields_autoplaced)
+  (global_label "C1" (shape input) (at 241.935 113.03 0) (fields_autoplaced)
     (effects (font (size 1.27 1.27)) (justify left))
-    (property "Intersheetrefs" "${INTERSHEET_REFS}" (at 246.8276 85.0106 0)
+    (property "Intersheetrefs" "${INTERSHEET_REFS}" (at 246.8276 112.9506 0)
       (effects (font (size 1.27 1.27)) (justify left) hide)
     )
   )
-  (global_label "C0" (shape input) (at 241.935 87.63 0) (fields_autoplaced)
+  (global_label "C0" (shape input) (at 241.935 118.11 0) (fields_autoplaced)
     (effects (font (size 1.27 1.27)) (justify left))
-    (property "Intersheetrefs" "${INTERSHEET_REFS}" (at 246.8276 87.5506 0)
+    (property "Intersheetrefs" "${INTERSHEET_REFS}" (at 246.8276 118.0306 0)
       (effects (font (size 1.27 1.27)) (justify left) hide)
     )
@@
     )
   )
-  (global_label "R2" (shape input) (at 241.935 118.11 0) (fields_autoplaced)
+  (global_label "R2" (shape input) (at 241.935 57.15 0) (fields_autoplaced)
     (effects (font (size 1.27 1.27)) (justify left))
-    (property "Intersheetrefs" "${INTERSHEET_REFS}" (at 246.8276 118.1894 0)
+    (property "Intersheetrefs" "${INTERSHEET_REFS}" (at 246.8276 57.2294 0)
       (effects (font (size 1.27 1.27)) (justify left) hide)
     )
@@
     )
   )
+  (symbol (lib_id "Device:C") (at 242.57 31.75 0) (unit 1)
+    (in_bom yes) (on_board yes) (dnp no) (fields_autoplaced)
+    (property "Reference" "C9" (at 246.38 30.4799 0)
+      (effects (font (size 1.27 1.27)) (justify left))
+    )
+    (property "Value" "1µ" (at 246.38 33.0199 0)
+      (effects (font (size 1.27 1.27)) (justify left))
+    )
+    (property "Footprint" "Capacitor_SMD:C_0805_2012Metric_Pad1.18x1.45mm_HandSolder" (at 243.5352 35.56 0)
+      (effects (font (size 1.27 1.27)) hide)
+    )
+    (property "Datasheet" "~" (at 242.57 31.75 0)
+      (effects (font (size 1.27 1.27)) hide)
+    )
+    (pin "1")
+    (pin "2")
+    (instances
+      (project "acacia-2"
+        (path "/c5eaf993-5ca3-41a9-9f58-50b86c0038a2"
+          (reference "C9") (unit 1)
+        )
+      )
+    )
+  )
   (symbol (lib_id "Device:D") (at 140.97 48.895 90) (unit 1)
     (in_bom yes) (on_board yes) (dnp no)
@@
         )
       )
+    )
+  )
+  (symbol (lib_id "power:GNDD") (at 242.57 36.83 0) (unit 1)
+    (in_bom yes) (on_board yes) (dnp no)
+    (property "Reference" "#PWR040" (at 242.57 43.18 0)
+      (effects (font (size 1.27 1.27)) hide)
+    )
+    (property "Value" "GNDD" (at 242.57 40.64 0)
+      (effects (font (size 1.27 1.27)))
+    )
+    (property "Footprint" "" (at 242.57 36.83 0)
+      (effects (font (size 1.27 1.27)) hide)
+    )
+    (property "Datasheet" "" (at 242.57 36.83 0)
+      (effects (font (size 1.27 1.27)) hide)
+    )
+    (pin "1")
+    (instances
+      (project "acacia-2"
+        (path "/c5eaf993-5ca3-41a9-9f58-50b86c0038a2"
+          (reference "#PWR040") (unit 1)
+        )
+      )
