File: acacia/kicad/acacia-2.kicad_sch (KiCad schematic)
At the start: 124 parts, among them J1 GroveMiniTrack, J2 TM040040, J3 USB4105-GF-A-060, SW1 Q, SW10 P, SW11 A, SW12 S, SW13 D, SW14 F, SW15 G, SW16 H, SW17 J, SW18 K, SW19 L, SW2 W, SW20 B, SW21 RESET, SW22 Z, SW23 X, SW24 C, SW25 V, SW26 Sft, SW27 Spc, SW28 N, SW29 M, SW3 E, SW30 Com, SW31 Dot, SW32 Tab, SW33 Prv, SW34 L1, SW35 AGr, SW36 Esc, SW37 Del, SW38 Nxt, SW39 Ent, SW4 R, SW5 T, SW6 Y, SW7 U, SW8 I, SW9 O, U1 ATmega32U4-A, U2 USBLC6-2SC6, Y1 16MHz

Commit message: V2 gerber
Parts:
- D39, D40, D41, D42, D43, D44: footprint LED_SMD:LED_SK6805_PLCC4_2.4x2.7mm_P1.3mm -> LED_SMD:LED_SK6812_EC15_1.5x1.5mm
Changed lines of the file:
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@@
       (effects (font (size 1.27 1.27)))
     )
-    (property "Footprint" "LED_SMD:LED_SK6805_PLCC4_2.4x2.7mm_P1.3mm" (at 59.69 114.935 0)
+    (property "Footprint" "LED_SMD:LED_SK6812_EC15_1.5x1.5mm" (at 59.69 114.935 0)
       (effects (font (size 1.27 1.27)) (justify left top) hide)
     )
@@
       (effects (font (size 1.27 1.27)))
     )
-    (property "Footprint" "LED_SMD:LED_SK6805_PLCC4_2.4x2.7mm_P1.3mm" (at 84.455 114.935 0)
+    (property "Footprint" "LED_SMD:LED_SK6812_EC15_1.5x1.5mm" (at 84.455 114.935 0)
       (effects (font (size 1.27 1.27)) (justify left top) hide)
     )
@@
       (effects (font (size 1.27 1.27)))
     )
-    (property "Footprint" "LED_SMD:LED_SK6805_PLCC4_2.4x2.7mm_P1.3mm" (at 134.62 114.935 0)
+    (property "Footprint" "LED_SMD:LED_SK6812_EC15_1.5x1.5mm" (at 134.62 114.935 0)
       (effects (font (size 1.27 1.27)) (justify left top) hide)
     )
@@
       (effects (font (size 1.27 1.27)))
     )
-    (property "Footprint" "LED_SMD:LED_SK6805_PLCC4_2.4x2.7mm_P1.3mm" (at 160.655 114.935 0)
+    (property "Footprint" "LED_SMD:LED_SK6812_EC15_1.5x1.5mm" (at 160.655 114.935 0)
       (effects (font (size 1.27 1.27)) (justify left top) hide)
     )
@@
       (effects (font (size 1.27 1.27)))
     )
-    (property "Footprint" "LED_SMD:LED_SK6805_PLCC4_2.4x2.7mm_P1.3mm" (at 34.925 114.935 0)
+    (property "Footprint" "LED_SMD:LED_SK6812_EC15_1.5x1.5mm" (at 34.925 114.935 0)
       (effects (font (size 1.27 1.27)) (justify left top) hide)
     )
@@
       (effects (font (size 1.27 1.27)))
     )
-    (property "Footprint" "LED_SMD:LED_SK6805_PLCC4_2.4x2.7mm_P1.3mm" (at 108.585 114.935 0)
+    (property "Footprint" "LED_SMD:LED_SK6812_EC15_1.5x1.5mm" (at 108.585 114.935 0)
       (effects (font (size 1.27 1.27)) (justify left top) hide)
     )

Commit message: testing delimiter together
Other:
- note added: "MISSING PULLUPS"
